File: Wearable sports tracker/_autosave-Embedded Processing.kicad_sch (KiCad schematic)
At the start: 7 parts, among them U1 STM32WB55RGVx

Commit message: ORDER TO MAKE CONCEPTION
Parts:
- added C7: 4u7, symbol Device:C
- added C8, C9: 100n, symbol Device:C
- C6: value 100n -> 4u7
Connections:
- net GND: now also U1.32 (VSSRF), U1.42 (VSSSMPS), U1.69 (VSS), C7.2, C8.2, C9.2
- net +3.3V: now reaches C1.1, C2.1, C3.1, C4.1, C5.1, C6.1, U1.1 (VBAT), U1.14 (VDDA), U1.30 (VDD), U1.45 (VDD), U1.55 (VDDUSB), U1.68 (VDD)
- net +3.3V: now also U1.33 (VDDRF), U1.44 (VDDSMPS), C7.1, C8.1, C9.1
