File: Wearable sports tracker/Wearable sports tracker.kicad_sch (KiCad schematic)
At the start: 1 part, among them U1 STM32WB55RGVx

Commit message: Nothing important
Parts:
- removed U1: STM32WB55RGVx, Package_DFN_QFN:QFN-68-1EP_8x8mm_P0.4mm_EP6.4x6.4mm, symbol MCU_ST_STM32WB:STM32WB55RGVx
Other:
- added sheet Embedded Processing (Embedded Processing.kicad_sch)
- added sheet Signal Acquisition Sensor (Signal Acquisition Sensor.kicad_sch)
- added sheet Transmision & Stockage (untitled.kicad_sch)
- note added: "Embedded Processing"
- note added: "Signal Acquisition Sensor"
- note added: "Supply Voltage & Battery management"
- note added: "Transmision & Stockage"

Commit message: MCU HSE & LSE Crystals
Other:
- company: (none) -> VAR.SYSTEMS
- title: (none) ->  Wearable Sports Tracker
Changed lines of the file:
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@@
 	(generator_version "9.0")
 	(paper "A4")
+	(title_block
+		(title " Wearable Sports Tracker")
+		(date "2025-11-09")
+		(company "VAR.SYSTEMS")
+		(comment 1 "Francisco VARELA")
+	)
 	(text "Signal Acquisition Sensor"
 		(exclude_from_sim no)
