File: Wearable sports tracker/untitled.kicad_sch (KiCad schematic)
At the start: 0 parts

Commit message: RF section
Parts:
- added C13: 0.8pF, symbol Device:C
- added C14: 0.3pF, symbol Device:C
- added FLT1: ~, VARELA:FIL_DEA160915LT-1169, symbol VARELA:DLF162500LT-5028A1
- added J1: Conn_Coaxial, symbol Connector:Conn_Coaxial
- added L3: 2.7nH, symbol Device:L
Connections:
- new net GND: C13.2, C14.2, FLT1.2 (GND), FLT1.4 (GND), J1.2 (Ext)
- new net RF1: C13.1, L3.1
- new net RF_ANT: FLT1.3 (OUT), J1.1 (In)
- new net RF_MATCH: C14.1, FLT1.1 (IN), L3.2
